File: variable_clock_module/variable_clock_module.kicad_sch (KiCad schematic)
At the start: 4 parts, among them IC1 ICM7555ISA+T, IC2 ICM7555ISA+T, IC3 ICM7555ISA+T

Commit message: minor changes
Parts:
- removed IC2, IC3: ICM7555ISA+T, SOIC127P600X175-8N, symbol SamacSys_Parts:ICM7555ISA+T
- added R?: ESR03EZPJ152, RESC1608X55N, symbol SamacSys_Parts:ESR03EZPJ152
Connections:
- net GND: now reaches IC1.1 (GND)
- net VCC: now reaches IC1.8 (V+)
Other:
- moved on the sheet: IC1, VR1
